File: Enhanced/PROTO2/C1581.kicad_pcb (KiCad board)
At the start: 2 copper layers, 183.9 x 111.3 mm, 80 parts, among them CN1 FLOPPY POWER, CN2 FLOPPY, CN3 IEC, CN4 IEC, CN5 LEDS, CN6 DIN-4, CN7 INTERNAL IEC, CN8 EXTERNAL POWER, CN9 XLEDS, J1 PIN34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

Commit message: Add EMI component values
Add missing EMI component values and generated new Interactive BOMs for both Enhanced and Internal Proto2 designs.
Parts:
- EM1, EM2, EM3, EM4: value EMI -> 100pf
- FB1, FB2, FB3, FB4, FB5, FB6: value R -> FB
Changed lines of the file:
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@@
 			)
 		)
-		(property "Value" "R"
+		(property "Value" "FB"
 			(at 6.35 2.72 90)
 			(layer "F.Fab")
@@
 			)
 		)
-		(property "Value" "R"
+		(property "Value" "FB"
 			(at 6.35 2.72 90)
 			(layer "F.Fab")
@@
 			)
 		)
-		(property "Value" "EMI"
+		(property "Value" "100pf"
 			(at 0 7.41 90)
 			(layer "F.Fab")
@@
 			)
 		)
-		(property "Value" "EMI"
+		(property "Value" "100pf"
 			(at 0 7.41 90)
 			(layer "F.Fab")
@@
 			)
 		)
-		(property "Value" "EMI"
+		(property "Value" "100pf"
 			(at 0 7.41 90)
 			(layer "F.Fab")
@@
 			)
 		)
-		(property "Value" "R"
+		(property "Value" "FB"
 			(at 6.35 2.72 90)
 			(layer "F.Fab")
@@
 			)
 		)
-		(property "Value" "R"
+		(property "Value" "FB"
 			(at 6.35 2.72 90)
 			(layer "F.Fab")
@@
 			)
 		)
-		(property "Value" "R"
+		(property "Value" "FB"
 			(at 6.35 2.72 0)
 			(layer "F.Fab")
@@
 			)
 		)
-		(property "Value" "R"
+		(property "Value" "FB"
 			(at 6.35 2.72 90)
 			(layer "F.Fab")
@@
 			)
 		)
-		(property "Value" "EMI"
+		(property "Value" "100pf"
 			(at 0 7.41 90)
 			(layer "F.Fab")
