File: Enhanced/PROTO2/C1581.kicad_sch (KiCad schematic)
At the start: 80 parts, among them CN1 FLOPPY POWER, CN2 FLOPPY, CN3 IEC, CN4 IEC, CN5 LEDS, CN6 DIN-4, CN7 INTERNAL IEC, CN8 EXTERNAL POWER, CN9 XLEDS, J1 PIN34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

Commit message: Add EMI component values
Add missing EMI component values and generated new Interactive BOMs for both Enhanced and Internal Proto2 designs.
Parts:
- EM1, EM2, EM3, EM4: value EMI -> 100pf
- FB1, FB2, FB3, FB4, FB5, FB6: value R -> FB
Other:
- note added: "UPDATED: 2025-11-29"
- note removed: "UPDATED: 2025-09-17"
Changed lines of the file:
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@@
 		)
 	)
-	(text "UPDATED: 2025-09-17"
+	(text "UPDATED: 2025-11-29"
 		(exclude_from_sim no)
 		(at 13.462 283.972 0)
@@
 			)
 		)
-		(property "Value" "R"
+		(property "Value" "FB"
 			(at 55.753 61.6966 0)
 			(effects
@@
 			)
 		)
-		(property "Value" "EMI"
+		(property "Value" "100pf"
 			(at 377.0122 179.4002 0)
 			(effects
@@
 			)
 		)
-		(property "Value" "R"
+		(property "Value" "FB"
 			(at 100.838 190.5 0)
 			(effects
@@
 			)
 		)
-		(property "Value" "EMI"
+		(property "Value" "100pf"
 			(at 377.5202 132.0292 0)
 			(effects
@@
 			)
 		)
-		(property "Value" "R"
+		(property "Value" "FB"
 			(at 62.738 180.34 0)
 			(effects
@@
 			)
 		)
-		(property "Value" "EMI"
+		(property "Value" "100pf"
 			(at 377.5202 147.7772 0)
 			(effects
@@
 			)
 		)
-		(property "Value" "R"
+		(property "Value" "FB"
 			(at 52.578 170.942 0)
 			(effects
@@
 			)
 		)
-		(property "Value" "R"
+		(property "Value" "FB"
 			(at 103.378 180.34 0)
 			(effects
@@
 			)
 		)
-		(property "Value" "R"
+		(property "Value" "FB"
 			(at 55.753 55.3466 0)
 			(effects
@@
 			)
 		)
-		(property "Value" "EMI"
+		(property "Value" "100pf"
 			(at 377.1392 163.6522 0)
 			(effects
